File: cnote.brd (EAGLE design)
At the start: 100 x 100 mm, 9 parts

Commit message: Fixed connector part number
Parts:
- U$1: value WURTH_WR-TBL-2418-6 -> WURTH_WR-TBL-2416-6; device travis:WURTH_WR-TBL-2418-6 -> travis:WURTH_WR-TBL-2416-6
Changed lines of the file:
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@@
 <?xml version="1.0" encoding="utf-8"?>
 <!DOCTYPE eagle SYSTEM "eagle.dtd">
-<eagle version="9.1.3">
+<eagle version="9.2.2">
 <drawing>
 <settings>
@@
 <attribute name="NAME" x="38.1" y="95.25" size="2.54" layer="25"/>
 </element>
-<element name="U$1" library="travis" package="WURTH_WR-TBL-2418-6" value="WURTH_WR-TBL-2418-6" x="3.81" y="50.8" rot="R90"/>
+<element name="U$1" library="travis" package="WURTH_WR-TBL-2416-6" value="WURTH_WR-TBL-2416-6" x="3.81" y="50.8" smashed="yes" rot="R90"/>
 </elements>
 <signals>
